File: ORCA_CORE/_autosave-usp.kicad_sch (KiCad schematic)
At the start: 15 parts, among them U11 AP64502

Commit message: making usp
Parts:
- added C29: 0.01u, symbol Device:C
- added R23, R24: 100k, symbol Device:R
Connections:
- net at U11.4 (RT/CLK): now also R23.1
- net at U11.6 (SS): now also C29.1
- new net: R23.2, R24.1
Changed lines of the file:
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@@
+    (stroke (width 0) (type default))
+  )
+  (wire (pts (xy 116.84 54.61) (xy 116.84 52.07))
     (stroke (width 0) (type default))
   )
@@
     (stroke (width 0) (type default))
   )
+  (wire (pts (xy 116.84 52.07) (xy 123.19 52.07))
+    (stroke (width 0) (type default))
+  )
   (wire (pts (xy 73.66 43.18) (xy 73.66 49.53))
     (stroke (width 0) (type default))
@@
     (stroke (width 0) (type default))
   )
+  (wire (pts (xy 107.95 49.53) (xy 123.19 49.53))
+    (stroke (width 0) (type default))
+  )
   (wire (pts (xy 90.17 128.27) (xy 90.17 124.46))
     (stroke (width 0) (type default))
@@
   )
   (wire (pts (xy 43.18 146.05) (xy 43.18 143.51))
+    (stroke (width 0) (type default))
+  )
+  (wire (pts (xy 107.95 50.8) (xy 107.95 49.53))
     (stroke (width 0) (type default))
   )
@@
     )
   )
+  (symbol (lib_id "Device:C") (at 116.84 58.42 0) (unit 1)
+    (in_bom yes) (on_board yes) (dnp no) (fields_autoplaced)
+    (property "Reference" "C29" (at 120.65 57.15 0)
+      (effects (font (size 1.27 1.27)) (justify left))
+    )
+    (property "Value" "0.01u" (at 120.65 59.69 0)
+      (effects (font (size 1.27 1.27)) (justify left))
+    )
+    (property "Footprint" "" (at 117.8052 62.23 0)
+      (effects (font (size 1.27 1.27)) hide)
+    )
+    (property "Datasheet" "~" (at 116.84 58.42 0)
+      (effects (font (size 1.27 1.27)) hide)
+    )
+    (pin "2")
+    (pin "1")
+    (instances
+      (project "ORCA_CORE"
+        (path "/895d6bb7-4008-488b-a34b-0077e9f7e4a1/6a7faaf2-e424-4dfa-bbc5-1df218d33dea"
+          (reference "C29") (unit 1)
+        )
+      )
+    )
+  )
   (symbol (lib_id "Device:C") (at 69.85 43.18 90) (unit 1)
     (in_bom yes) (on_board yes) (dnp no)
@@
     )
   )
+  (symbol (lib_id "Device:R") (at 107.95 54.61 0) (unit 1)
+    (in_bom yes) (on_board yes) (dnp no) (fields_autoplaced)
+    (property "Reference" "R23" (at 110.49 53.34 0)
+      (effects (font (size 1.27 1.27)) (justify left))
+    )
+    (property "Value" "100k" (at 110.49 55.88 0)
+      (effects (font (size 1.27 1.27)) (justify left))
+    )
+    (property "Footprint" "" (at 106.172 54.61 90)
+      (effects (font (size 1.27 1.27)) hide)
+    )
+    (property "Datasheet" "~" (at 107.95 54.61 0)
+      (effects (font (size 1.27 1.27)) hide)
+    )
+    (pin "2")
+    (pin "1")
+    (instances
+      (project "ORCA_CORE"
+        (path "/895d6bb7-4008-488b-a34b-0077e9f7e4a1/6a7faaf2-e424-4dfa-bbc5-1df218d33dea"
+          (reference "R23") (unit 1)
+        )
+      )
+    )
+  )
   (symbol (lib_id "Device:C") (at 43.18 149.86 0) (unit 1)
     (in_bom yes) (on_board yes) (dnp no) (fields_autoplaced)
@@
         )
       )
+    )
+  )
+  (symbol (lib_id "Device:R") (at 107.95 62.23 0) (unit 1)
+    (in_bom yes) (on_board yes) (dnp no) (fields_autoplaced)
+    (property "Reference" "R24" (at 110.49 60.96 0)
+      (effects (font (size 1.27 1.27)) (justify left))
+    )
+    (property "Value" "100k" (at 110.49 63.5 0)
+      (effects (font (size 1.27 1.27)) (justify left))
+    )
+    (property "Footprint" "" (at 106.172 62.23 90)
+      (effects (font (size 1.27 1.27)) hide)
+    )
+    (property "Datasheet" "~" (at 107.95 62.23 0)
+      (effects (font (size 1.27 1.27)) hide)
+    )
+    (pin "2")
+    (pin "1")
+    (instances
+      (project "ORCA_CORE"
+        (path "/895d6bb7-4008-488b-a34b-0077e9f7e4a1/6a7faaf2-e424-4dfa-bbc5-1df218d33dea"
+          (reference "R24") (unit 1)
+        )
+      )
