File: ORCA_CORE/power.kicad_sch (KiCad schematic)
At the start: 67 parts, among them J4 emergence, Q1 TJ60S04M3L, Q2 BSS138, Q3 BSS138, Q4 IRLML6402, U1 LTC2301IMS, U2 NJM78055DL1, U4 RH1B-UDC6V, U5 TPH11006NL, U6 TPH11006NL, U7 NJW4860, U8 AZ1117-3.3

Commit message: plate power
Parts:
- removed R5, R6: 2.2k, Resistor_SMD:R_0603_1608Metric_Pad0.98x0.95mm_HandSolder, symbol Device:R
- added H1, H2, H3, H4: Hole_power, MountingHole:MountingHole_3.2mm_M3, symbol Mechanical:MountingHole
Connections:
- net +6V_power: no longer C22.1, C23.2, Q1.1 (D), R1.2
- net +BATT_power: now also C22.2, C23.2, Q1.1 (D), R1.2
- net GND: now also C22.1; no longer C22.2
Other:
- moved on the sheet: C22
