File: ORCA_CORE/power.kicad_sch (KiCad schematic)
At the start: 69 parts, among them J4 emergence, Q1 TJ60S04M3L, Q2 BSS138, Q3 BSS138, Q4 IRLML6402, U1 LTC2301IMS, U2 NJM78055DL1, U4 RH1B-UDC6V, U5 TPH11006NL, U6 TPH11006NL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

Commit message: plate all parts
Parts:
- added R50: 2.2k, Resistor_SMD:R_0603_1608Metric_Pad0.98x0.95mm_HandSolder, symbol Device:R
Connections:
- net GND: now also R50.1
- net emerge_order: now also R50.2
Changed lines of the file:
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@@
   (junction (at 149.86 40.64) (diameter 0) (color 0 0 0 0)
+  )
+  (junction (at 95.25 138.43) (diameter 0) (color 0 0 0 0)
   )
   (junction (at 40.64 40.64) (diameter 0) (color 0 0 0 0)
@@
     (stroke (width 0) (type default))
   )
+  (wire (pts (xy 95.25 138.43) (xy 100.33 138.43))
+    (stroke (width 0) (type default))
+  )
   (wire (pts (xy 250.19 22.86) (xy 252.73 22.86))
     (stroke (width 0) (type default))
@@
     (stroke (width 0) (type default))
   )
-  (wire (pts (xy 99.06 138.43) (xy 100.33 138.43))
+  (wire (pts (xy 91.44 138.43) (xy 95.25 138.43))
     (stroke (width 0) (type default))
   )
@@
     (effects (font (size 1.27 1.27)) (justify left))
   )
-  (hierarchical_label "emerge_order" (shape input) (at 99.06 138.43 180) (fields_autoplaced)
+  (hierarchical_label "emerge_order" (shape input) (at 91.44 138.43 180) (fields_autoplaced)
     (effects (font (size 1.27 1.27)) (justify right))
   )
@@
     )
   )
+  (symbol (lib_id "Device:R") (at 95.25 134.62 0) (unit 1)
+    (in_bom yes) (on_board yes) (dnp no) (fields_autoplaced)
+    (property "Reference" "R50" (at 97.79 133.35 0)
+      (effects (font (size 1.27 1.27)) (justify left))
+    )
+    (property "Value" "2.2k" (at 97.79 135.89 0)
+      (effects (font (size 1.27 1.27)) (justify left))
+    )
+    (property "Footprint" "Resistor_SMD:R_0603_1608Metric_Pad0.98x0.95mm_HandSolder" (at 93.472 134.62 90)
+      (effects (font (size 1.27 1.27)) hide)
+    )
+    (property "Datasheet" "~" (at 95.25 134.62 0)
+      (effects (font (size 1.27 1.27)) hide)
+    )
+    (pin "2")
+    (pin "1")
+    (instances
+      (project "ORCA_CORE"
+        (path "/895d6bb7-4008-488b-a34b-0077e9f7e4a1/62c40b6d-2f8c-4265-a550-d6ec27759bcd"
+          (reference "R50") (unit 1)
+        )
+      )
+    )
+  )
   (symbol (lib_id "Device:R") (at 154.94 113.03 0) (unit 1)
     (in_bom yes) (on_board yes) (dnp no) (fields_autoplaced)
@@
         )
       )
+    )
+  )
+  (symbol (lib_id "power:GND") (at 95.25 130.81 180) (unit 1)
+    (in_bom yes) (on_board yes) (dnp no) (fields_autoplaced)
+    (property "Reference" "#PWR033" (at 95.25 124.46 0)
+      (effects (font (size 1.27 1.27)) hide)
+    )
+    (property "Value" "GND" (at 95.25 125.73 0)
+      (effects (font (size 1.27 1.27)))
+    )
+    (property "Footprint" "" (at 95.25 130.81 0)
+      (effects (font (size 1.27 1.27)) hide)
+    )
+    (property "Datasheet" "" (at 95.25 130.81 0)
+      (effects (font (size 1.27 1.27)) hide)
+    )
+    (pin "1")
+    (instances
+      (project "ORCA_CORE"
+        (path "/895d6bb7-4008-488b-a34b-0077e9f7e4a1/62c40b6d-2f8c-4265-a550-d6ec27759bcd"
+          (reference "#PWR033") (unit 1)
+        )
+      )

Commit message: change extern lib path to project dir
Parts:
- U4: footprint Relay_THT:RH1-U -> relay:RH1-U
Changed lines of the file:
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@@
       (effects (font (size 1.27 1.27)))
     )
-    (property "Footprint" "Relay_THT:RH1-U" (at 127 90.17 0)
+    (property "Footprint" "relay:RH1-U" (at 127 90.17 0)
       (effects (font (size 1.27 1.27)) hide)
     )

Commit message: placed an order
Parts:
- R19: value 10 -> 360
