File: ORCA_CORE/ORCA_CORE.kicad_sch (KiCad schematic)
At the start: 11 parts, among them J1 data_line_power, J17 Vin_motor, J18 data_line_power, J19 +5Vout_cpu, J2 I2C_power, J3 Vout_motor, J5 Vin_batt, J6 Vin_ex, J7 Vout_power2usp, J8 Vin_power2usp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

Commit message: plate power and usp
Parts:
- J19: value +5Vout_cpu -> +5Vin_cpu
Connections:
- net GND: no longer J19.1 (Pin_1), J9.1 (Pin_1)
- new net GND1: J19.1 (Pin_1), J9.1 (Pin_1)
Other:
- sheet cpu ports: added GND_5V; removed none
- sheet usp ports: added GND_5V; removed none
Changed lines of the file:
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@@
     (stroke (width 0) (type default))
   )
-  (symbol (lib_id "power:GND") (at 67.31 106.68 270) (unit 1)
-    (in_bom yes) (on_board yes) (dnp no) (fields_autoplaced)
-    (property "Reference" "#PWR069" (at 60.96 106.68 0)
-      (effects (font (size 1.27 1.27)) hide)
-    )
-    (property "Value" "GND" (at 63.5 106.68 90)
-      (effects (font (size 1.27 1.27)) (justify right))
-    )
-    (property "Footprint" "" (at 67.31 106.68 0)
-      (effects (font (size 1.27 1.27)) hide)
-    )
-    (property "Datasheet" "" (at 67.31 106.68 0)
-      (effects (font (size 1.27 1.27)) hide)
-    )
-    (pin "1")
-    (instances
-      (project "ORCA_CORE"
-        (path "/895d6bb7-4008-488b-a34b-0077e9f7e4a1"
-          (reference "#PWR069") (unit 1)
-        )
-      )
-    )
-  )
-  (symbol (lib_id "power:GND") (at 58.42 120.65 90) (unit 1)
-    (in_bom yes) (on_board yes) (dnp no) (fields_autoplaced)
-    (property "Reference" "#PWR070" (at 64.77 120.65 0)
-      (effects (font (size 1.27 1.27)) hide)
-    )
-    (property "Value" "GND" (at 62.23 120.65 90)
-      (effects (font (size 1.27 1.27)) (justify right))
-    )
-    (property "Footprint" "" (at 58.42 120.65 0)
-      (effects (font (size 1.27 1.27)) hide)
-    )
-    (property "Datasheet" "" (at 58.42 120.65 0)
+  (symbol (lib_id "power:GND") (at 58.42 116.84 90) (unit 1)
+    (in_bom yes) (on_board yes) (dnp no) (fields_autoplaced)
+    (property "Reference" "#PWR070" (at 64.77 116.84 0)
+      (effects (font (size 1.27 1.27)) hide)
+    )
+    (property "Value" "GND" (at 62.23 116.84 90)
+      (effects (font (size 1.27 1.27)) (justify right))
+    )
+    (property "Footprint" "" (at 58.42 116.84 0)
+      (effects (font (size 1.27 1.27)) hide)
+    )
+    (property "Datasheet" "" (at 58.42 116.84 0)
       (effects (font (size 1.27 1.27)) hide)
     )
@@
         (path "/895d6bb7-4008-488b-a34b-0077e9f7e4a1"
           (reference "#PWR070") (unit 1)
+        )
+      )
+    )
+  )
+  (symbol (lib_id "power:GND1") (at 82.55 109.22 90) (unit 1)
+    (in_bom yes) (on_board yes) (dnp no) (fields_autoplaced)
+    (property "Reference" "#PWR05" (at 88.9 109.22 0)
+      (effects (font (size 1.27 1.27)) hide)
+    )
+    (property "Value" "GND1" (at 86.36 109.22 90)
+      (effects (font (size 1.27 1.27)) (justify right))
+    )
+    (property "Footprint" "" (at 82.55 109.22 0)
+      (effects (font (size 1.27 1.27)) hide)
+    )
+    (property "Datasheet" "" (at 82.55 109.22 0)
+      (effects (font (size 1.27 1.27)) hide)
+    )
+    (pin "1")
+    (instances
+      (project "ORCA_CORE"
+        (path "/895d6bb7-4008-488b-a34b-0077e9f7e4a1"
+          (reference "#PWR05") (unit 1)
         )
       )
@@
     )
   )
-  (symbol (lib_id "power:GND") (at 82.55 109.22 90) (unit 1)
-    (in_bom yes) (on_board yes) (dnp no) (fields_autoplaced)
-    (property "Reference" "#PWR0105" (at 88.9 109.22 0)
-      (effects (font (size 1.27 1.27)) hide)
-    )
-    (property "Value" "GND" (at 86.36 109.22 90)
-      (effects (font (size 1.27 1.27)) (justify right))
-    )
-    (property "Footprint" "" (at 82.55 109.22 0)
-      (effects (font (size 1.27 1.27)) hide)
-    )
-    (property "Datasheet" "" (at 82.55 109.22 0)
-      (effects (font (size 1.27 1.27)) hide)
-    )
-    (pin "1")
-    (instances
-      (project "ORCA_CORE"
-        (path "/895d6bb7-4008-488b-a34b-0077e9f7e4a1"
-          (reference "#PWR0105") (unit 1)
+  (symbol (lib_id "power:GND1") (at 138.43 123.19 0) (unit 1)
+    (in_bom yes) (on_board yes) (dnp no) (fields_autoplaced)
+    (property "Reference" "#PWR026" (at 138.43 129.54 0)
+      (effects (font (size 1.27 1.27)) hide)
+    )
+    (property "Value" "GND1" (at 138.43 128.27 0)
+      (effects (font (size 1.27 1.27)))
+    )
+    (property "Footprint" "" (at 138.43 123.19 0)
+      (effects (font (size 1.27 1.27)) hide)
+    )
+    (property "Datasheet" "" (at 138.43 123.19 0)
+      (effects (font (size 1.27 1.27)) hide)
+    )
+    (pin "1")
+    (instances
+      (project "ORCA_CORE"
+        (path "/895d6bb7-4008-488b-a34b-0077e9f7e4a1"
+          (reference "#PWR026") (unit 1)
         )
       )
@@
     )
   )
+  (symbol (lib_id "power:GND1") (at 67.31 106.68 270) (unit 1)
+    (in_bom yes) (on_board yes) (dnp no) (fields_autoplaced)
+    (property "Reference" "#PWR030" (at 60.96 106.68 0)
+      (effects (font (size 1.27 1.27)) hide)
+    )
+    (property "Value" "GND1" (at 63.5 106.68 90)
+      (effects (font (size 1.27 1.27)) (justify right))
+    )
+    (property "Footprint" "" (at 67.31 106.68 0)
+      (effects (font (size 1.27 1.27)) hide)
+    )
+    (property "Datasheet" "" (at 67.31 106.68 0)
+      (effects (font (size 1.27 1.27)) hide)
+    )
+    (pin "1")
+    (instances
+      (project "ORCA_CORE"
+        (path "/895d6bb7-4008-488b-a34b-0077e9f7e4a1"
+          (reference "#PWR030") (unit 1)
+        )
+      )
+    )
+  )
+  (symbol (lib_id "power:GND1") (at 194.31 173.99 0) (unit 1)
+    (in_bom yes) (on_board yes) (dnp no) (fields_autoplaced)
+    (property "Reference" "#PWR031" (at 194.31 180.34 0)
+      (effects (font (size 1.27 1.27)) hide)
+    )
+    (property "Value" "GND1" (at 194.31 179.07 0)
+      (effects (font (size 1.27 1.27)))
+    )
+    (property "Footprint" "" (at 194.31 173.99 0)
+      (effects (font (size 1.27 1.27)) hide)
+    )
+    (property "Datasheet" "" (at 194.31 173.99 0)
+      (effects (font (size 1.27 1.27)) hide)
+    )
+    (pin "1")
+    (instances
+      (project "ORCA_CORE"
+        (path "/895d6bb7-4008-488b-a34b-0077e9f7e4a1"
+          (reference "#PWR031") (unit 1)
+        )
+      )
+    )
+  )
   (symbol (lib_id "Connector_Generic:Conn_01x02") (at 91.44 29.21 180) (unit 1)
     (in_bom yes) (on_board yes) (dnp no)
@@
     )
   )
+  (symbol (lib_id "power:PWR_FLAG") (at 194.31 173.99 0) (unit 1)
+    (in_bom yes) (on_board yes) (dnp no) (fields_autoplaced)
+    (property "Reference" "#FLG016" (at 194.31 172.085 0)
+      (effects (font (size 1.27 1.27)) hide)
+    )
+    (property "Value" "PWR_FLAG" (at 194.31 169.799 0)
+      (effects (font (size 1.27 1.27)))
+    )
+    (property "Footprint" "" (at 194.31 173.99 0)
+      (effects (font (size 1.27 1.27)) hide)
+    )
+    (property "Datasheet" "~" (at 194.31 173.99 0)
+      (effects (font (size 1.27 1.27)) hide)
+    )
+    (pin "1")
+    (instances
+      (project "ORCA_CORE"
+        (path "/895d6bb7-4008-488b-a34b-0077e9f7e4a1"
+          (reference "#FLG016") (unit 1)
+        )
+      )
+    )
+  )
   (symbol (lib_id "power:GND") (at 63.5 95.25 0) (unit 1)
     (in_bom yes) (on_board yes) (dnp no) (fields_autoplaced)
@@
         (path "/895d6bb7-4008-488b-a34b-0077e9f7e4a1"
           (reference "#PWR054") (unit 1)
+        )
+      )
+    )
+  )
+  (symbol (lib_id "power:GND1") (at 58.42 120.65 90) (unit 1)
+    (in_bom yes) (on_board yes) (dnp no) (fields_autoplaced)
+    (property "Reference" "#PWR029" (at 64.77 120.65 0)
+      (effects (font (size 1.27 1.27)) hide)
+    )
+    (property "Value" "GND1" (at 62.23 120.65 90)
+      (effects (font (size 1.27 1.27)) (justify right))
+    )
+    (property "Footprint" "" (at 58.42 120.65 0)
+      (effects (font (size 1.27 1.27)) hide)
+    )
+    (property "Datasheet" "" (at 58.42 120.65 0)
+      (effects (font (size 1.27 1.27)) hide)
+    )
+    (pin "1")
+    (instances
+      (project "ORCA_CORE"
+        (path "/895d6bb7-4008-488b-a34b-0077e9f7e4a1"
+          (reference "#PWR029") (unit 1)
         )
       )
@@
       (effects (font (size 1.27 1.27)) (justify left))
     )
-    (property "Value" "+5Vout_cpu" (at 87.63 102.87 0)
+    (property "Value" "+5Vin_cpu" (at 87.63 102.87 0)
       (effects (font (size 1.27 1.27)) (justify left))
     )
@@
       (effects (font (size 1.27 1.27)) (justify left top))
     )
-    (pin "GND" output (at 58.42 120.65 0)
+    (pin "GND" output (at 58.42 116.84 0)
       (effects (font (size 1.27 1.27)) (justify right))
     )
@@
     )
     (pin "Vout" input (at 58.42 109.22 0)
+      (effects (font (size 1.27 1.27)) (justify right))
+    )
+    (pin "GND_5V" output (at 58.42 120.65 0)
       (effects (font (size 1.27 1.27)) (justify right))
     )
@@
       (effects (font (size 1.27 1.27)) (justify left))
     )
+    (pin "GND_5V" bidirectional (at 138.43 123.19 270)
+      (effects (font (size 1.27 1.27)) (justify left))
+    )

Commit message: complete wireing and filling usp
Connections:
- net GND1: no longer J19.1 (Pin_1)
- new net GND2: J19.1 (Pin_1)
Changed lines of the file:
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@@
-    )
-  )
-  (symbol (lib_id "power:GND1") (at 82.55 109.22 90) (unit 1)
-    (in_bom yes) (on_board yes) (dnp no) (fields_autoplaced)
-    (property "Reference" "#PWR05" (at 88.9 109.22 0)
-      (effects (font (size 1.27 1.27)) hide)
-    )
-    (property "Value" "GND1" (at 86.36 109.22 90)
-      (effects (font (size 1.27 1.27)) (justify right))
-    )
-    (property "Footprint" "" (at 82.55 109.22 0)
-      (effects (font (size 1.27 1.27)) hide)
-    )
-    (property "Datasheet" "" (at 82.55 109.22 0)
-      (effects (font (size 1.27 1.27)) hide)
-    )
-    (pin "1")
-    (instances
-      (project "ORCA_CORE"
-        (path "/895d6bb7-4008-488b-a34b-0077e9f7e4a1"
-          (reference "#PWR05") (unit 1)
-        )
-      )
     )
   )
@@
     )
   )
-  (symbol (lib_id "power:GND1") (at 138.43 123.19 0) (unit 1)
-    (in_bom yes) (on_board yes) (dnp no) (fields_autoplaced)
-    (property "Reference" "#PWR026" (at 138.43 129.54 0)
-      (effects (font (size 1.27 1.27)) hide)
-    )
-    (property "Value" "GND1" (at 138.43 128.27 0)
-      (effects (font (size 1.27 1.27)))
-    )
-    (property "Footprint" "" (at 138.43 123.19 0)
-      (effects (font (size 1.27 1.27)) hide)
-    )
-    (property "Datasheet" "" (at 138.43 123.19 0)
-      (effects (font (size 1.27 1.27)) hide)
-    )
-    (pin "1")
-    (instances
-      (project "ORCA_CORE"
-        (path "/895d6bb7-4008-488b-a34b-0077e9f7e4a1"
-          (reference "#PWR026") (unit 1)
-        )
-      )
-    )
-  )
   (symbol (lib_id "Connector_Generic:Conn_01x03") (at 85.09 58.42 0) (unit 1)
     (in_bom yes) (on_board yes) (dnp no)
@@
     )
   )
+  (symbol (lib_id "power:PWR_FLAG") (at 204.47 173.99 0) (unit 1)
+    (in_bom yes) (on_board yes) (dnp no) (fields_autoplaced)
+    (property "Reference" "#FLG017" (at 204.47 172.085 0)
+      (effects (font (size 1.27 1.27)) hide)
+    )
+    (property "Value" "PWR_FLAG" (at 204.47 169.799 0)
+      (effects (font (size 1.27 1.27)))
+    )
+    (property "Footprint" "" (at 204.47 173.99 0)
+      (effects (font (size 1.27 1.27)) hide)
+    )
+    (property "Datasheet" "~" (at 204.47 173.99 0)
+      (effects (font (size 1.27 1.27)) hide)
+    )
+    (pin "1")
+    (instances
+      (project "ORCA_CORE"
+        (path "/895d6bb7-4008-488b-a34b-0077e9f7e4a1"
+          (reference "#FLG017") (unit 1)
+        )
+      )
+    )
+  )
   (symbol (lib_id "Connector_Generic:Conn_01x02") (at 91.44 29.21 180) (unit 1)
     (in_bom yes) (on_board yes) (dnp no)
@@
     )
   )
+  (symbol (lib_id "power:GND2") (at 204.47 173.99 0) (unit 1)
+    (in_bom yes) (on_board yes) (dnp no) (fields_autoplaced)
+    (property "Reference" "#PWR026" (at 204.47 180.34 0)
+      (effects (font (size 1.27 1.27)) hide)
+    )
+    (property "Value" "GND2" (at 204.47 179.07 0)
+      (effects (font (size 1.27 1.27)))
+    )
+    (property "Footprint" "" (at 204.47 173.99 0)
+      (effects (font (size 1.27 1.27)) hide)
+    )
+    (property "Datasheet" "" (at 204.47 173.99 0)
+      (effects (font (size 1.27 1.27)) hide)
+    )
+    (pin "1")
+    (instances
+      (project "ORCA_CORE"
+        (path "/895d6bb7-4008-488b-a34b-0077e9f7e4a1"
+          (reference "#PWR026") (unit 1)
+        )
+      )
+    )
+  )
+  (symbol (lib_id "power:GND2") (at 82.55 109.22 90) (unit 1)
+    (in_bom yes) (on_board yes) (dnp no) (fields_autoplaced)
+    (property "Reference" "#PWR05" (at 88.9 109.22 0)
+      (effects (font (size 1.27 1.27)) hide)
+    )
+    (property "Value" "GND2" (at 86.36 109.22 90)
+      (effects (font (size 1.27 1.27)) (justify right))
+    )
+    (property "Footprint" "" (at 82.55 109.22 0)
+      (effects (font (size 1.27 1.27)) hide)
+    )
+    (property "Datasheet" "" (at 82.55 109.22 0)
+      (effects (font (size 1.27 1.27)) hide)
+    )
+    (pin "1")
+    (instances
+      (project "ORCA_CORE"
+        (path "/895d6bb7-4008-488b-a34b-0077e9f7e4a1"
+          (reference "#PWR05") (unit 1)
+        )
+      )
+    )
+  )
   (symbol (lib_id "Connector_Generic:Conn_01x02") (at 22.86 43.18 180) (unit 1)
     (in_bom yes) (on_board yes) (dnp no) (fields_autoplaced)
@@
         )
       )
+    )
+  )
+  (symbol (lib_id "power:GND2") (at 138.43 123.19 0) (unit 1)
+    (in_bom yes) (on_board yes) (dnp no) (fields_autoplaced)
+    (property "Reference" "#PWR025" (at 138.43 129.54 0)
+      (effects (font (size 1.27 1.27)) hide)
+    )
+    (property "Value" "GND2" (at 138.43 128.27 0)
+      (effects (font (size 1.27 1.27)))
+    )
+    (property "Footprint" "" (at 138.43 123.19 0)
+      (effects (font (size 1.27 1.27)) hide)
+    )
+    (property "Datasheet" "" (at 138.43 123.19 0)
+      (effects (font (size 1.27 1.27)) hide)
+    )
+    (pin "1")
+    (instances
+      (project "ORCA_CORE"
+        (path "/895d6bb7-4008-488b-a34b-0077e9f7e4a1"
+          (reference "#PWR025") (unit 1)
+        )
+      )
