File: ORCA_CORE/ORCA_CORE.kicad_sch (KiCad schematic)
At the start: 22 parts, among them J18 +6V_motor, J19 +5Vin_cpu, J23 md_arm, J24 md_fork, J25 servo_arm, J33 cpu_female_left, J34 cpu_female_right, J35 hat_male_right, J36 enable_arm, J37 enable_arm, J38 servo_arm, J39 md_arm, J40 md_fork, J41 cpu_male_left, J42 uart, J43 uart_device, J45 reset, J46 reset, J47 led, J48 led, J51 usb_A_device, J52 usb_A

Commit message: most of wire placed. try update kicad to use replicate library
Connections:
- net +3V3: no longer J23.6 (Pin_6), J24.6 (Pin_6), J25.6 (Pin_6), J35.19 (Pin_19), J41.2 (Pin_2), J46.2 (Pin_2)
- net +5V: no longer J35.2 (Pin_2), J41.3 (Pin_3), J42.4 (Pin_4), J47.2 (Pin_2)
- net arm/GND_cpu renamed arm/GND_arm
- net arm/Vin_cpu renamed arm/Vin_arm
- net cpu/emerg_detector renamed cpu/emerge_detector
- net md_arm/GND_cpu renamed md_arm/GND_md
- net md_arm/Vin_cpu renamed md_arm/Vin_md
- net md_fork/GND_cpu renamed md_fork/GND_md
- net md_fork/Vin_cpu renamed md_fork/Vin_md
- new net Vin_3V3_cpu_hat: J23.6 (Pin_6), J24.6 (Pin_6), J25.6 (Pin_6), J35.19 (Pin_19), J41.2 (Pin_2), J46.2 (Pin_2)
- new net Vin_cpu_hat: J35.2 (Pin_2), J41.3 (Pin_3), J42.4 (Pin_4), J47.2 (Pin_2)
Other:
- sheet arm ports: added GND_arm, Vin_arm; removed GND_cpu, Vin_cpu
- sheet cpu ports: added emerge_detector; removed emerg_detector
- sheet md_arm ports: added GND_md, Vin_md; removed GND_cpu, Vin_cpu
- sheet md_fork ports: added GND_md, Vin_md; removed GND_cpu, Vin_cpu
