File: ORCA_CORE/ORCA_CORE.kicad_sch (KiCad schematic)
At the start: 22 parts, among them J18 +6V_motor, J19 +5Vin_cpu, J23 md_arm, J24 md_fork, J25 servo_arm, J33 cpu_female_left, J34 cpu_female_right, J35 hat_male_right, J36 enable_arm, J37 enable_arm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

Commit message: end wiring
Changed lines of the file:
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@@
-			)
-		)
-		(pin "TXD_5V" input
-			(at 90.17 34.29 0)
-			(effects
-				(font
-					(size 1.27 1.27)
-				)
-				(justify right)
 			)
 		)
@@
 			(effects
 				(font
+					(size 1.27 1.27)
+				)
+				(justify right)
+			)
+		)
+		(pin "TXD_5V" output
+			(at 90.17 34.29 0)
+			(effects
+				(font
