File: ORCA_CORE/usp.kicad_sch (KiCad schematic)
At the start: 52 parts, among them J21 Conn_01x02, Q5 TJ60S04M3L, U10 HY2112, U11 AP64502, U12 TPS61230A__board, U3 CN3058E, U9 FS8205

Commit message: change extern lib path to project dir
Parts:
- J21: footprint Battery:BatteryHolder_1xAA_code -> battery_case:BatteryHolder_1xAA_code
- L1: footprint Inductor_SMD:L_12x12mm_H8mm_withmodel -> inductor:L_12x12mm_H8mm_withmodel
- U12: footprint Converter_DCDC:TPS61230A -> converter_module:TPS61230A
Changed lines of the file:
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@@
       (effects (font (size 1.27 1.27)) (justify left))
     )
-    (property "Footprint" "Battery:BatteryHolder_1xAA_code" (at 252.73 105.41 0)
+    (property "Footprint" "battery_case:BatteryHolder_1xAA_code" (at 252.73 105.41 0)
       (effects (font (size 1.27 1.27)) hide)
     )
@@
       (effects (font (size 1.27 1.27)))
     )
-    (property "Footprint" "Converter_DCDC:TPS61230A" (at 246.38 34.29 0)
+    (property "Footprint" "converter_module:TPS61230A" (at 246.38 34.29 0)
       (effects (font (size 1.27 1.27)) hide)
     )
@@
       (effects (font (size 1.27 1.27)))
     )
-    (property "Footprint" "Inductor_SMD:L_12x12mm_H8mm_withmodel" (at 170.18 36.83 0)
-      (effects (font (size 1.27 1.27)) hide)
-    )
+    (property "Footprint" "inductor:L_12x12mm_H8mm_withmodel" (at 170.18 36.83 0)
+      (effects (font (size 1.27 1.27)) hide)
+    )
