File: ORCA_CORE/cpu.kicad_sch (KiCad schematic)
At the start: 59 parts, among them J10 Raspberry_Pi_2_3, J11 wheel_left, J44 servo_camera, J8 wheel_front, J9 wheel_right, Q1 BSS138, Q2 BSS138, Q8 BSS138, U14 BNO055, U18 TLP293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

Commit message: most of wire placed. try update kicad to use replicate library
Connections:
- net emerg_detector is gone; now on net emerge_detector: R52.1
- net emerge_detector: no longer J10.15 (GPIO22), U19.3
- net emerge_order: no longer J10.18 (GPIO24), R55.1
- net power_checker: no longer J10.16 (GPIO23), U18.3
- net LED12: no longer names the net of U2.19 (LED12)
- net LED13: no longer names the net of U2.20 (LED13)
- net LED14: no longer names the net of U2.21 (LED14)
- net LED15: no longer names the net of U2.22 (LED15)
- new net emerge_detector_out: J10.15 (GPIO22), U19.3
- new net emerge_order_in: J10.18 (GPIO24), R55.1
- new net power_checker_out: J10.16 (GPIO23), U18.3
- no-connect marks 17 -> 21

Commit message: complete almost all wires. add mouse coms sensor
Parts:
- removed H10, H22: Hole_cup, MountingHole:MountingHole_3.2mm_M3, symbol Mechanical:MountingHole
- removed H21, H9: Hole_cpu, MountingHole:MountingHole_3.2mm_M3, symbol Mechanical:MountingHole
- added U26: ~, mouse_sensor:PMW3360, symbol mylib:PMW3360
Connections:
- net GND1: no longer U14.7 (GND)
- no-connect marks 21 -> 22

Commit message: end wiring
Parts:
- removed U14: BNO055, IMU:BNO055_short, symbol mylib:BNO055
- added C13: 0.1u, Capacitor_SMD:C_0603_1608Metric_Pad1.08x0.95mm_HandSolder, symbol Device:C
- added C14: 10u, Capacitor_SMD:C_1206_3216Metric_Pad1.33x1.80mm_HandSolder, symbol Device:C
- added R57: 1.2k, Resistor_SMD:R_0603_1608Metric_Pad0.98x0.95mm_HandSolder, symbol Device:R
- added R58: 2k, Resistor_SMD:R_0603_1608Metric_Pad0.98x0.95mm_HandSolder, symbol Device:R
- added R74: 2.2k, Resistor_SMD:R_0603_1608Metric_Pad0.98x0.95mm_HandSolder, symbol Device:R
- R72: value 2.2k -> 10k
- U26: value ~ -> PMW3360
Connections:
- net SCL_cpu is gone; now on net SCL: J10.5 (SCL/GPIO3)
- net SDA_cpu is gone; now on net SDA: J10.3 (SDA/GPIO2)
- net +3V3: now also R73.2, U26.5 (VDDIO), R57.2, R74.2; no longer R72.1, R73.1
- net GND1: now also U26.8 (GND), C13.1, C14.1, R58.1
- net SCL: now also R74.1; no longer R73.2
- net SDA: now also R73.1; no longer R72.2
- net MOSI: now reaches J10.19 (MOSI0/GPIO10)
- net MOSI: now also U26.11 (MOSI)
- net MISO: now reaches J10.21 (MISO0/GPIO9)
- net MISO: now also U26.12 (MISO)
- net SCLK: now reaches J10.23 (SCLK0/GPIO11)
- net SCLK: now also U26.9 (MOTION)
- net CS0: now reaches J10.24 (~{CE0}/GPIO8)
- net CS0: now also U26.13 (NCS)
- net at U26.15 (LED_P): now also R72.1, U26.4 (VDD), R57.1, R58.2
- net at U26.3 (VDDPIX): now also C13.2, C14.2
- net at U26.7 (NRESET): now also R72.2
- no-connect marks 22 -> 20
Other:
- moved on the sheet: Q1, Q2, Q8, R34, R4, R5, R6, R7, R8, R9, U2, U26
