File: ORCA_CORE/_autosave-external_io.kicad_sch (KiCad schematic)
At the start: 27 parts, among them J1 Vext_in, J2 6Vout, J3 6Vout, J4 6Vout, J5 6Vin, J50 USB_A, J6 Vext_out, J7 6Vout, P1 USB_C_Receptacle_USB2.0, SW2 REST_sw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

Commit message: complete all CORE board. knew that 2 boards cannot be wrote in 1 sketch
Parts:
- J2: footprint Conn:AMASS_XT30U-F_Vertical_withmodel_male -> Conn:power_pad
- J3, J4, J7: footprint Conn:AMASS_XT30U-F_Vertical_withmodel_male -> Connector_JST:JST_XH_B2B-XH-A_1x02_P2.50mm_Vertical
- J50: footprint Connector_USB:USB_A_Kycon_KUSBX-AS1N-B_Horizontal -> Conn:TypeA_connector_KUSBX-AS1N-B
Changed lines of the file:
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@@
 			)
 		)
-		(property "Footprint" "Conn:AMASS_XT30U-F_Vertical_withmodel_male"
+		(property "Footprint" "Conn:power_pad"
 			(at 212.09 40.64 0)
 			(effects
@@
 			)
 		)
-		(property "Footprint" "Conn:AMASS_XT30U-F_Vertical_withmodel_male"
+		(property "Footprint" "Connector_JST:JST_XH_B2B-XH-A_1x02_P2.50mm_Vertical"
 			(at 231.14 40.64 0)
 			(effects
@@
 			)
 		)
-		(property "Footprint" "Conn:AMASS_XT30U-F_Vertical_withmodel_male"
+		(property "Footprint" "Connector_JST:JST_XH_B2B-XH-A_1x02_P2.50mm_Vertical"
 			(at 218.44 40.64 0)
 			(effects
@@
 			)
 		)
-		(property "Footprint" "Connector_USB:USB_A_Kycon_KUSBX-AS1N-B_Horizontal"
+		(property "Footprint" "Conn:TypeA_connector_KUSBX-AS1N-B"
 			(at 217.17 134.62 0)
 			(effects
@@
 			)
 		)
-		(property "Footprint" "Conn:AMASS_XT30U-F_Vertical_withmodel_male"
+		(property "Footprint" "Connector_JST:JST_XH_B2B-XH-A_1x02_P2.50mm_Vertical"
 			(at 224.79 40.64 0)
 			(effects
